File: 150x90mm_80_degree_angle/kicad.9/7_segment_digit/7_segment_digit.kicad_sch (KiCad schematic)
At the start: 10 parts, among them X1 PLS-10

Commit message: Добавил символ и посадочную площадку СИД SMD 5050. Обновил схему и ПП.
Parts:
- removed D1: LED, LED_THT:LED_D5.0mm, symbol Device:LED
- added D1: ~, led_strip:LED_SMD_5050_6, symbol 7_segment_digit:Diode
- LS1, LS2, LS3, LS4, LS5, LS6, LS7: footprint led_strip:led_strip_50mm_len_8mm_height_TH -> led_strip:led_strip_50mm_len_8mm_height
Connections:
- net 1: now also D1.2 (K0), D1.4 (K1), D1.6 (K2)
- net VCC: now also D1.1 (A0), D1.3 (A1), D1.5 (A2)
Changed lines of the file:
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@@
+	)
+	(junction
+		(at 187.96 120.65)
+		(diameter 0)
+		(color 0 0 0 0)
+	)
+	(junction
+		(at 180.34 120.65)
+		(diameter 0)
+		(color 0 0 0 0)
 	)
 	(junction
@@
 	(wire
 		(pts
+			(xy 187.96 120.65) (xy 187.96 124.46)
+		)
+		(stroke
+			(width 0)
+			(type default)
+		)
+	)
+	(wire
+		(pts
+			(xy 180.34 116.84) (xy 180.34 120.65)
+		)
+		(stroke
+			(width 0)
+			(type default)
+		)
+	)
+	(wire
+		(pts
 			(xy 140.97 59.69) (xy 140.97 55.88)
 		)
@@
 	(wire
 		(pts
+			(xy 180.34 120.65) (xy 180.34 124.46)
+		)
+		(stroke
+			(width 0)
+			(type default)
+		)
+	)
+	(wire
+		(pts
 			(xy 175.26 67.31) (xy 170.18 67.31)
 		)
@@
 		(pts
 			(xy 161.29 107.95) (xy 163.83 107.95)
+		)
+		(stroke
+			(width 0)
+			(type default)
+		)
+	)
+	(wire
+		(pts
+			(xy 187.96 116.84) (xy 187.96 120.65)
 		)
 		(stroke
@@
 			)
 		)
-		(property "Footprint" "led_strip:led_strip_50mm_len_8mm_height_TH"
+		(property "Footprint" "led_strip:led_strip_50mm_len_8mm_height"
 			(at 152.4 82.55 0)
 			(effects
@@
 			)
 		)
-		(property "Footprint" "led_strip:led_strip_50mm_len_8mm_height_TH"
+		(property "Footprint" "led_strip:led_strip_50mm_len_8mm_height"
 			(at 152.4 54.61 0)
 			(effects
@@
 			)
 		)
-		(property "Footprint" "led_strip:led_strip_50mm_len_8mm_height_TH"
+		(property "Footprint" "led_strip:led_strip_50mm_len_8mm_height"
 			(at 139.7 95.25 0)
 			(effects
@@
 			)
 		)
-		(property "Footprint" "led_strip:led_strip_50mm_len_8mm_height_TH"
+		(property "Footprint" "led_strip:led_strip_50mm_len_8mm_height"
 			(at 139.7 68.58 0)
 			(effects
@@
 	)
 	(symbol
-		(lib_id "Device:LED")
-		(at 184.15 120.65 0)
-		(unit 1)
-		(exclude_from_sim no)
-		(in_bom yes)
-		(on_board yes)
-		(dnp no)
-		(property "Reference" "D1"
-			(at 184.15 117.856 0)
-			(effects
-				(font
-					(size 1.27 1.27)
-				)
-			)
-		)
-		(property "Value" "LED"
-			(at 183.896 123.952 0)
-			(effects
-				(font
-					(size 1.27 1.27)
-				)
-			)
-		)
-		(property "Footprint" "LED_THT:LED_D5.0mm"
-			(at 184.15 120.65 0)
-			(effects
-				(font
-					(size 1.27 1.27)
-				)
-				(hide yes)
-			)
-		)
-		(property "Datasheet" "~"
-			(at 184.15 120.65 0)
-			(effects
-				(font
-					(size 1.27 1.27)
-				)
-				(hide yes)
-			)
-		)
-		(property "Description" "Light emitting diode"
-			(at 184.15 120.65 0)
-			(effects
-				(font
-					(size 1.27 1.27)
-				)
-				(hide yes)
-			)
-		)
-		(property "Sim.Pins" "1=K 2=A"
-			(at 184.15 120.65 0)
-			(effects
-				(font
-					(size 1.27 1.27)
-				)
-				(hide yes)
-			)
-		)
-		(pin "1"
-		)
-		(pin "2"
-		)
-		(instances
-			(project ""
-				(path "/5df25448-ca4f-4e12-a809-76052196b894"
-					(reference "D1")
-					(unit 1)
-				)
-			)
-		)
-	)
-	(symbol
 		(lib_id "7_segment_digit:led_strip_50mm_len_8mm_height")
 		(at 165.1 68.58 90)
@@
 			)
 		)
-		(property "Footprint" "led_strip:led_strip_50mm_len_8mm_height_TH"
+		(property "Footprint" "led_strip:led_strip_50mm_len_8mm_height"
 			(at 165.1 68.58 0)
 			(effects
@@
 			)
 		)
-		(property "Footprint" "led_strip:led_strip_50mm_len_8mm_height_TH"
+		(property "Footprint" "led_strip:led_strip_50mm_len_8mm_height"
 			(at 152.4 109.22 0)
 			(effects
@@
 			)
 		)
-		(property "Footprint" "led_strip:led_strip_50mm_len_8mm_height_TH"
+		(property "Footprint" "led_strip:led_strip_50mm_len_8mm_height"
 			(at 165.1 95.25 0)
 			(effects
@@
 					(unit 1)
 				)
+			)
+		)
+	)
+	(symbol
+		(lib_id "7_segment_digit:Diode")
+		(at 180.34 120.65 0)
+		(unit 1)
+		(exclude_from_sim no)
+		(in_bom yes)
+		(on_board yes)
+		(dnp no)
+		(fields_autoplaced yes)
+		(property "Reference" "D1"
+			(at 183.8325 111.76 0)
+			(effects
+				(font
+					(size 1.27 1.27)
+				)
+			)
+		)
+		(property "Value" "~"
+			(at 183.8325 114.3 0)
+			(effects
+				(font
+					(size 1.27 1.27)
+				)
+			)
+		)
+		(property "Footprint" "led_strip:LED_SMD_5050_6"
+			(at 180.34 120.65 0)
+			(effects
+				(font
+					(size 1.27 1.27)
+				)
+				(hide yes)
+			)
+		)
+		(property "Datasheet" ""
+			(at 180.34 120.65 0)
+			(effects
+				(font
+					(size 1.27 1.27)
+				)
+				(hide yes)
+			)
+		)
+		(property "Description" ""
+			(at 180.34 120.65 0)
+			(effects
+				(font
+					(size 1.27 1.27)
+				)
+				(hide yes)
+			)
+		)
+		(pin "3"
+		)
+		(pin "2"
+		)
+		(pin "6"
+		)
+		(pin "5"
+		)
+		(pin "1"
+		)
+		(pin "4"
+		)
+		(instances
+			(project ""
+				(path "/5df25448-ca4f-4e12-a809-76052196b894"
+					(reference "D1")
+					(unit 1)
+				)
